File: hardware/cad/B2/ethernet_1.kicad_sch (KiCad schematic)
At the start: 8 parts, among them U3 W5500

Commit message: Update Site source
Parts:
- C21, C22, C23: footprint Capacitor_SMD:C_0603_1608Metric -> Capacitor_SMD:C_0402_1005Metric; symbol Rack:C100n -> Rack:C100n_0402; LCSC C14663 -> C1525; MPN CC0603KRX7R9BB104 -> CL05B104KO5NNNC
Changed lines of the file:
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@@
 (wire(pts(xy 50.8 168.91)(xy 53.34 168.91))(stroke(width 0)(type default)))
 (global_label "GND_CTRL"(shape bidirectional)(at 53.34 168.91 0)(effects(font(size 1.016 1.016))(justify left))(property "Intersheetrefs" "${INTERSHEET_REFS}"(at 53.34 168.91 0)(effects(font(size 1 1))(hide yes))))
-(symbol(lib_id "Rack:C100n")(at 146.05 168.91 0)(unit 1)(exclude_from_sim no)(in_bom yes)(on_board yes)(dnp no)(property "Reference" "C21"(at 146.05 162.64 0)(effects(font(size 1.016 1.016))))(property "Value" "100n"(at 146.05 165.14 0)(effects(font(size 1.016 1.016))))(property "Footprint" "Capacitor_SMD:C_0603_1608Metric"(at 146.05 168.91 0)(effects(font(size 1.016 1.016))(hide yes)))(property "LCSC" "C14663"(at 146.05 168.91 0)(effects(font(size 1.016 1.016))(hide yes)))(property "MPN" "CC0603KRX7R9BB104"(at 146.05 168.91 0)(effects(font(size 1.016 1.016))(hide yes)))(pin "1")(pin "2")(instances(project "rack-atx-controller"(path "/e26e9c9a-6137-5b0e-b3e3-ffc5633a6c0f/1331d7f0-0c80-53a9-bf95-e086def53a7b"(reference "C21")(unit 1)))))
+(symbol(lib_id "Rack:C100n_0402")(at 146.05 168.91 0)(unit 1)(exclude_from_sim no)(in_bom yes)(on_board yes)(dnp no)(property "Reference" "C21"(at 146.05 162.64 0)(effects(font(size 1.016 1.016))))(property "Value" "100n"(at 146.05 165.14 0)(effects(font(size 1.016 1.016))))(property "Footprint" "Capacitor_SMD:C_0402_1005Metric"(at 146.05 168.91 0)(effects(font(size 1.016 1.016))(hide yes)))(property "LCSC" "C1525"(at 146.05 168.91 0)(effects(font(size 1.016 1.016))(hide yes)))(property "MPN" "CL05B104KO5NNNC"(at 146.05 168.91 0)(effects(font(size 1.016 1.016))(hide yes)))(pin "1")(pin "2")(instances(project "rack-atx-controller"(path "/e26e9c9a-6137-5b0e-b3e3-ffc5633a6c0f/1331d7f0-0c80-53a9-bf95-e086def53a7b"(reference "C21")(unit 1)))))
 (wire(pts(xy 140.97 168.91)(xy 138.43 168.91))(stroke(width 0)(type default)))
 (global_label "3V3_ETH_A"(shape bidirectional)(at 138.43 168.91 180)(effects(font(size 1.016 1.016))(justify right))(property "Intersheetrefs" "${INTERSHEET_REFS}"(at 138.43 168.91 0)(effects(font(size 1 1))(hide yes))))
 (wire(pts(xy 151.13 168.91)(xy 153.67 168.91))(stroke(width 0)(type default)))
 (global_label "GND_CTRL"(shape bidirectional)(at 153.67 168.91 0)(effects(font(size 1.016 1.016))(justify left))(property "Intersheetrefs" "${INTERSHEET_REFS}"(at 153.67 168.91 0)(effects(font(size 1 1))(hide yes))))
-(symbol(lib_id "Rack:C100n")(at 246.38 168.91 0)(unit 1)(exclude_from_sim no)(in_bom yes)(on_board yes)(dnp no)(property "Reference" "C22"(at 246.38 162.64 0)(effects(font(size 1.016 1.016))))(property "Value" "100n"(at 246.38 165.14 0)(effects(font(size 1.016 1.016))))(property "Footprint" "Capacitor_SMD:C_0603_1608Metric"(at 246.38 168.91 0)(effects(font(size 1.016 1.016))(hide yes)))(property "LCSC" "C14663"(at 246.38 168.91 0)(effects(font(size 1.016 1.016))(hide yes)))(property "MPN" "CC0603KRX7R9BB104"(at 246.38 168.91 0)(effects(font(size 1.016 1.016))(hide yes)))(pin "1")(pin "2")(instances(project "rack-atx-controller"(path "/e26e9c9a-6137-5b0e-b3e3-ffc5633a6c0f/1331d7f0-0c80-53a9-bf95-e086def53a7b"(reference "C22")(unit 1)))))
+(symbol(lib_id "Rack:C100n_0402")(at 246.38 168.91 0)(unit 1)(exclude_from_sim no)(in_bom yes)(on_board yes)(dnp no)(property "Reference" "C22"(at 246.38 162.64 0)(effects(font(size 1.016 1.016))))(property "Value" "100n"(at 246.38 165.14 0)(effects(font(size 1.016 1.016))))(property "Footprint" "Capacitor_SMD:C_0402_1005Metric"(at 246.38 168.91 0)(effects(font(size 1.016 1.016))(hide yes)))(property "LCSC" "C1525"(at 246.38 168.91 0)(effects(font(size 1.016 1.016))(hide yes)))(property "MPN" "CL05B104KO5NNNC"(at 246.38 168.91 0)(effects(font(size 1.016 1.016))(hide yes)))(pin "1")(pin "2")(instances(project "rack-atx-controller"(path "/e26e9c9a-6137-5b0e-b3e3-ffc5633a6c0f/1331d7f0-0c80-53a9-bf95-e086def53a7b"(reference "C22")(unit 1)))))
 (wire(pts(xy 241.3 168.91)(xy 238.76 168.91))(stroke(width 0)(type default)))
 (global_label "3V3_ETH_A"(shape bidirectional)(at 238.76 168.91 180)(effects(font(size 1.016 1.016))(justify right))(property "Intersheetrefs" "${INTERSHEET_REFS}"(at 238.76 168.91 0)(effects(font(size 1 1))(hide yes))))
 (wire(pts(xy 251.46 168.91)(xy 254.0 168.91))(stroke(width 0)(type default)))
 (global_label "GND_CTRL"(shape bidirectional)(at 254.0 168.91 0)(effects(font(size 1.016 1.016))(justify left))(property "Intersheetrefs" "${INTERSHEET_REFS}"(at 254.0 168.91 0)(effects(font(size 1 1))(hide yes))))
-(symbol(lib_id "Rack:C100n")(at 345.44 168.91 0)(unit 1)(exclude_from_sim no)(in_bom yes)(on_board yes)(dnp no)(property "Reference" "C23"(at 345.44 162.64 0)(effects(font(size 1.016 1.016))))(property "Value" "100n"(at 345.44 165.14 0)(effects(font(size 1.016 1.016))))(property "Footprint" "Capacitor_SMD:C_0603_1608Metric"(at 345.44 168.91 0)(effects(font(size 1.016 1.016))(hide yes)))(property "LCSC" "C14663"(at 345.44 168.91 0)(effects(font(size 1.016 1.016))(hide yes)))(property "MPN" "CC0603KRX7R9BB104"(at 345.44 168.91 0)(effects(font(size 1.016 1.016))(hide yes)))(pin "1")(pin "2")(instances(project "rack-atx-controller"(path "/e26e9c9a-6137-5b0e-b3e3-ffc5633a6c0f/1331d7f0-0c80-53a9-bf95-e086def53a7b"(reference "C23")(unit 1)))))
+(symbol(lib_id "Rack:C100n_0402")(at 345.44 168.91 0)(unit 1)(exclude_from_sim no)(in_bom yes)(on_board yes)(dnp no)(property "Reference" "C23"(at 345.44 162.64 0)(effects(font(size 1.016 1.016))))(property "Value" "100n"(at 345.44 165.14 0)(effects(font(size 1.016 1.016))))(property "Footprint" "Capacitor_SMD:C_0402_1005Metric"(at 345.44 168.91 0)(effects(font(size 1.016 1.016))(hide yes)))(property "LCSC" "C1525"(at 345.44 168.91 0)(effects(font(size 1.016 1.016))(hide yes)))(property "MPN" "CL05B104KO5NNNC"(at 345.44 168.91 0)(effects(font(size 1.016 1.016))(hide yes)))(pin "1")(pin "2")(instances(project "rack-atx-controller"(path "/e26e9c9a-6137-5b0e-b3e3-ffc5633a6c0f/1331d7f0-0c80-53a9-bf95-e086def53a7b"(reference "C23")(unit 1)))))
 (wire(pts(xy 340.36 168.91)(xy 337.82 168.91))(stroke(width 0)(type default)))
 (global_label "3V3_ETH_A"(shape bidirectional)(at 337.82 168.91 180)(effects(font(size 1.016 1.016))(justify right))(property "Intersheetrefs" "${INTERSHEET_REFS}"(at 337.82 168.91 0)(effects(font(size 1 1))(hide yes))))
