File: hardware/cad/B2/ethernet_2.kicad_sch (KiCad schematic)
At the start: 24 parts, among them J105 HR911105A, Y2 25MHz CL12pF

Commit message: Update Site source
Parts:
- C33: footprint Capacitor_SMD:C_0603_1608Metric -> Capacitor_SMD:C_0402_1005Metric; symbol Rack:C10n -> Rack:C10n_0402; LCSC C57112 -> C15195; MPN 0603B103K500NT -> CL05B103KB5NNNC
- C34, C35: footprint Capacitor_SMD:C_0603_1608Metric -> Capacitor_SMD:C_0402_1005Metric; symbol Rack:C6.8n -> Rack:C6.8n_0402; LCSC C1631 -> C318580; MPN 0603B682K500NT -> CL05B682KB5NNNC
- R20, R21: footprint Resistor_SMD:R_0603_1608Metric -> Resistor_SMD:R_0402_1005Metric; symbol Rack:R49.9 -> Rack:R49.9_0402; LCSC C23185 -> C25120; MPN 0603WAF499JT5E -> 0402WGF499JTCE
