File: hardware/cad/B2/processor_1.kicad_sch (KiCad schematic)
At the start: 10 parts, among them J104 TYPE-C-31-M-12, U2 ESP32-S3FN8

Commit message: Update Site source
Parts:
- U2: footprint Package_DFN_QFN:QFN-56-1EP_7x7mm_P0.4mm_EP4x4mm -> RackATX:ESP32_S3_QFN56_EP4_16Window
Changed lines of the file:
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@@
 (kicad_sch (version 20250114)(generator "eeschema")(paper "A3")(title_block (title "ESP32-S3FN8 / USB programming (1/2)")(rev "B.2")(company "Rack ATX Controller / ddasdkimo")(comment 1 "SCHEMATIC REVIEW - not a fabrication release"))
 (text "Wired Ethernet only. Leave LNA_IN open and never initialize Wi-Fi/BLE.\nGPIO26..32 used by internal quad flash: do not route. GPIO45 pulled low selects 3.3 V flash."(at 12 20 0)(effects(font(size 1.27 1.27))(justify left)))
-(symbol(lib_id "Rack:mcu")(at 54.61 92.71 0)(unit 1)(exclude_from_sim no)(in_bom yes)(on_board yes)(dnp no)(property "Reference" "U2"(at 54.61 49.60999999999999 0)(effects(font(size 1.016 1.016))))(property "Value" "ESP32-S3FN8"(at 54.61 52.10999999999999 0)(effects(font(size 1.016 1.016))))(property "Footprint" "Package_DFN_QFN:QFN-56-1EP_7x7mm_P0.4mm_EP4x4mm"(at 54.61 92.71 0)(effects(font(size 1.016 1.016))(hide yes)))(property "LCSC" "C2913196"(at 54.61 92.71 0)(effects(font(size 1.016 1.016))(hide yes)))(property "MPN" "ESP32-S3FN8"(at 54.61 92.71 0)(effects(font(size 1.016 1.016))(hide yes)))(pin "36")(pin "45")(pin "51")(pin "56")(pin "1")(pin "2")(pin "3")(pin "4")(pin "5")(pin "6")(pin "7")(pin "8")(pin "9")(pin "10")(pin "11")(pin "12")(pin "13")(pin "14")(pin "15")(pin "16")(pin "17")(pin "18")(pin "19")(pin "20")(pin "21")(pin "22")(pin "23")(pin "24")(pin "25")(pin "26")(pin "27")(pin "28")(pin "29")(pin "30")(pin "31")(pin "32")(pin "33")(pin "34")(pin "35")(pin "37")(pin "38")(pin "39")(pin "40")(pin "41")(pin "42")(pin "43")(pin "44")(pin "46")(pin "47")(pin "48")(pin "49")(pin "50")(pin "52")(pin "53")(pin "54")(pin "55")(pin "57")(instances(project "rack-atx-controller"(path "/e26e9c9a-6137-5b0e-b3e3-ffc5633a6c0f/9b65307c-93d4-5b24-8af6-c081e3e79102"(reference "U2")(unit 1)))))
+(symbol(lib_id "Rack:mcu")(at 54.61 92.71 0)(unit 1)(exclude_from_sim no)(in_bom yes)(on_board yes)(dnp no)(property "Reference" "U2"(at 54.61 49.60999999999999 0)(effects(font(size 1.016 1.016))))(property "Value" "ESP32-S3FN8"(at 54.61 52.10999999999999 0)(effects(font(size 1.016 1.016))))(property "Footprint" "RackATX:ESP32_S3_QFN56_EP4_16Window"(at 54.61 92.71 0)(effects(font(size 1.016 1.016))(hide yes)))(property "LCSC" "C2913196"(at 54.61 92.71 0)(effects(font(size 1.016 1.016))(hide yes)))(property "MPN" "ESP32-S3FN8"(at 54.61 92.71 0)(effects(font(size 1.016 1.016))(hide yes)))(pin "36")(pin "45")(pin "51")(pin "56")(pin "1")(pin "2")(pin "3")(pin "4")(pin "5")(pin "6")(pin "7")(pin "8")(pin "9")(pin "10")(pin "11")(pin "12")(pin "13")(pin "14")(pin "15")(pin "16")(pin "17")(pin "18")(pin "19")(pin "20")(pin "21")(pin "22")(pin "23")(pin "24")(pin "25")(pin "26")(pin "27")(pin "28")(pin "29")(pin "30")(pin "31")(pin "32")(pin "33")(pin "34")(pin "35")(pin "37")(pin "38")(pin "39")(pin "40")(pin "41")(pin "42")(pin "43")(pin "44")(pin "46")(pin "47")(pin "48")(pin "49")(pin "50")(pin "52")(pin "53")(pin "54")(pin "55")(pin "57")(instances(project "rack-atx-controller"(path "/e26e9c9a-6137-5b0e-b3e3-ffc5633a6c0f/9b65307c-93d4-5b24-8af6-c081e3e79102"(reference "U2")(unit 1)))))
 (wire(pts(xy 39.37 57.15)(xy 36.83 57.15))(stroke(width 0)(type default)))
 (global_label "ETH_RST_N"(shape bidirectional)(at 36.83 57.15 180)(effects(font(size 1.016 1.016))(justify right))(property "Intersheetrefs" "${INTERSHEET_REFS}"(at 36.83 57.15 0)(effects(font(size 1 1))(hide yes))))
