File: hardware/cad/B2/rack-atx-controller.kicad_sch (KiCad schematic)
At the start: 0 parts

Commit message: Update Site source
Other:
- note added: "B.2: ten hosts, POWER / RESET only. Original case LEDs remain on motherboard. 5 V input -> 3.3 V logic; ESP32-S3FN8 + W5500 -> 74HC595 -> twenty isolated dry contacts MC14541B counted timeout + independent ARM gate; no LED sensing or isolated DC/DC S.3 baseline / R.3 routing and package updates; factory DFM and prototype verification pending"
- note removed: "B.2: ten hosts, POWER / RESET only. Original case LEDs remain on motherboard. 5 V input -> 3.3 V logic; ESP32-S3FN8 + W5500 -> 74HC595 -> twenty isolated dry contacts MC14541B counted timeout + independent ARM gate; no LED sensing or isolated DC/DC S.3 compact layout; routing authorized after placement checks; no fabrication release"
