File: hardware/cad/B2/rack-atx-controller.kicad_pcb (KiCad board)
At the start: 2 copper layers, 100 x 110 mm, 304 parts, among them J01 S10B-PHDSS(LF)(SN), J02 S10B-PHDSS(LF)(SN), J03 S10B-PHDSS(LF)(SN), J04 S10B-PHDSS(LF)(SN), J05 S10B-PHDSS(LF)(SN), J06 S10B-PHDSS(LF)(SN), J07 S10B-PHDSS(LF)(SN), J08 S10B-PHDSS(LF)(SN), J09 S10B-PHDSS(LF)(SN), J10 S10B-PHDSS(LF)(SN), J101 WJ500V-5.08-2P, J102 PZ254V-11-02P, J103 PZ254V-11-02P, J104 TYPE-C-31-M-12, J105 HR911105A, Q1 AO3401A, Q10 MMBT3904, Q11 MMBT3904, Q12 MMBT3904, Q13 MMBT3904, Q14 MMBT3904, Q15 MMBT3904, Q16 MMBT3904, Q17 MMBT3904, Q18 MMBT3904, Q19 MMBT3904, Q2 MMBT3904, Q20 MMBT3904, Q200 MMBT3904, Q21 MMBT3904, Q22 MMBT3904, Q23 MMBT3904, Q24 MMBT3904, Q3 MMBT3904, Q4 AO3401A, Q5 MMBT3904, Q6 MMBT3904, Q7 MMBT3904, Q8 MMBT3904, Q9 MMBT3904, U1 AP63203WU-7, U10 TLP3122A(TPL,E, U11 TLP3122A(TPL,E, U12 TLP3122A(TPL,E, U13 TLP3122A(TPL,E, U14 TLP3122A(TPL,E, U15 TLP3122A(TPL,E, U16 TLP3122A(TPL,E, U17 TLP3122A(TPL,E, U18 TLP3122A(TPL,E, U19 TLP3122A(TPL,E, U2 ESP32-S3FN8, U20 TLP3122A(TPL,E, U21 TLP3122A(TPL,E, U22 TLP3122A(TPL,E, U23 TLP3122A(TPL,E, U24 TLP3122A(TPL,E, U25 TLP3122A(TPL,E, U26 TLP3122A(TPL,E, U27 TLP3122A(TPL,E, U3 W5500, U4 74HC595D,118, U5 74HC595D,118, U6 74HC595D,118, U7 MC14541BDR2G, U8 TLP3122A(TPL,E, U9 TLP3122A(TPL,E, Y1 40MHz CL12pF, Y2 25MHz CL12pF

Commit message: Update Site source
Parts:
- C21, C22, C23, C33, C34, C35: footprint Capacitor_SMD:C_0603_1608Metric -> Capacitor_SMD:C_0402_1005Metric
- R20, R21: footprint Resistor_SMD:R_0603_1608Metric -> Resistor_SMD:R_0402_1005Metric
- U2: footprint Package_DFN_QFN:QFN-56-1EP_7x7mm_P0.4mm_EP4x4mm -> RackATX:ESP32_S3_QFN56_EP4_16Window
- moved R8 30.7 mm to (12.5, 73.3), turned to 0 degrees
- moved R9 29.1 mm to (16.0, 73.3), turned to 0 degrees
- moved C34 11.8 mm to (24.1, 50.4), turned to 90 degrees
- moved C35 10.8 mm to (24.1, 46.7), turned to 180 degrees
- moved R18 9.95 mm to (26.6, 45.6), turned to 0 degrees
- moved C33 8.44 mm to (24.3, 48.5), turned to 90 degrees
- moved R21 6.98 mm to (25.9, 47.8), turned to 180 degrees
- moved R20 6.84 mm to (25.9, 49.2), turned to 180 degrees
- moved R25 3.01 mm to (39.5, 65.8), turned to 0 degrees
- moved R19 2.24 mm to (28.0, 42.5), turned to 90 degrees
- moved R26 1.53 mm to (43.0, 65.8), turned to 0 degrees
- moved C22 1.51 mm to (27.9, 49.8)
- moved C21 1.27 mm to (27.9, 47.5)
- moved C23 1.13 mm to (27.9, 51.2)
- moved R14 0.70 mm to (27.0, 53.2)
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Routing:
- net 3V3: track 290.0 -> 519.4 mm, vias 10 -> 21
- net OUT_LATCH: track 51.9 -> 154.2 mm, vias 4 -> 7
- net DRV_04: track 46.3 -> 134.2 mm
- net OUT_OE_N: track 126.3 -> 195.8 mm, vias 5 -> 11
- net DRV_08: track 57.7 -> 123.0 mm, vias 2 -> 4
- net DRV_03: track 56.0 -> 103.9 mm
- net TIMER_ARM: track 21.5 -> 66.8 mm
- net DRV_05: track 125.5 -> 85.6 mm, vias 2 -> 12
- net DRV_02: track 61.3 -> 94.0 mm, vias 2 -> 6
- net USB_CC2: track 37.7 -> 7.53 mm, vias 2 -> 0
- net USB_CC1: track 37.3 -> 9.59 mm
- net DRV_01: track 58.2 -> 85.5 mm, vias 2 -> 4
- net RJ_RD_N: track 25.8 -> 5.54 mm
- net ETH_RX_TERM: track 32.7 -> 13.4 mm, vias 2 -> 1
- net USB_VBUS_SENSE: track 20.9 -> 38.6 mm, vias 2 -> 4
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
Commit message: Update Site source
Other:
- board text added: "+"
- board text added: "-"
- board text added: "5V IN"
- board text added: "BOOT"
- board text added: "J01"
- board text added: "J02"
- board text added: "J03"
- board text added: "J04"
- board text added: "J05"
- board text added: "J06"
- board text added: "J07"
- board text added: "J08"
- board text added: "J09"
- board text added: "J10"
- board text added: "LAN"
- board text added: "MCU RST"
- board text added: "RACK ATX R3"
- board text added: "USB"
Changed lines of the file:
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@@
 		(layer "Edge.Cuts")
+	)
+	(gr_text "USB"
+		(at 4.7 62.5 0)
+		(layer "F.SilkS")
+		(effects
+			(font
+				(size 1 1)
+				(thickness 0.15)
+			)
+		)
 	)
 	(gr_text "3V3"
@@
 		)
 	)
+	(gr_text "LAN"
+		(at 10 39.5 0)
+		(layer "F.SilkS")
+		(effects
+			(font
+				(size 1 1)
+				(thickness 0.15)
+			)
+		)
+	)
 	(gr_text "PWR"
 		(at 11 26.55 0)
@@
 		)
 	)
+	(gr_text "5V IN"
+		(at 94 55 0)
+		(layer "F.SilkS")
+		(effects
+			(font
+				(size 1 1)
+				(thickness 0.15)
+			)
+		)
+	)
 	(gr_text "RST"
 		(at 11 83.45 180)
@@
 		)
 	)
+	(gr_text "J01"
+		(at 14 22 0)
+		(layer "F.SilkS")
+		(effects
+			(font
+				(size 1.2 1.2)
+				(thickness 0.15)
+			)
+		)
+	)
+	(gr_text "J06"
+		(at 14 88 0)
+		(layer "F.SilkS")
+		(effects
+			(font
+				(size 1.2 1.2)
+				(thickness 0.15)
+			)
+		)
+	)
+	(gr_text "J02"
+		(at 32 22 0)
+		(layer "F.SilkS")
+		(effects
+			(font
+				(size 1.2 1.2)
+				(thickness 0.15)
+			)
+		)
+	)
+	(gr_text "J07"
+		(at 32 88 0)
+		(layer "F.SilkS")
+		(effects
+			(font
+				(size 1.2 1.2)
+				(thickness 0.15)
+			)
+		)
+	)
+	(gr_text "J03"
+		(at 50 22 0)
+		(layer "F.SilkS")
+		(effects
+			(font
+				(size 1.2 1.2)
+				(thickness 0.15)
+			)
+		)
+	)
+	(gr_text "J08"
+		(at 50 88 0)
+		(layer "F.SilkS")
+		(effects
+			(font
+				(size 1.2 1.2)
+				(thickness 0.15)
+			)
+		)
+	)
+	(gr_text "J04"
+		(at 68 22 0)
+		(layer "F.SilkS")
+		(effects
+			(font
+				(size 1.2 1.2)
+				(thickness 0.15)
+			)
+		)
+	)
+	(gr_text "J09"
+		(at 68 88 0)
+		(layer "F.SilkS")
+		(effects
+			(font
+				(size 1.2 1.2)
+				(thickness 0.15)
+			)
+		)
+	)
+	(gr_text "J05"
+		(at 86 22 0)
+		(layer "F.SilkS")
+		(effects
+			(font
+				(size 1.2 1.2)
+				(thickness 0.15)
+			)
+		)
+	)
+	(gr_text "J10"
+		(at 86 88 0)
+		(layer "F.SilkS")
+		(effects
+			(font
+				(size 1.2 1.2)
+				(thickness 0.15)
+			)
+		)
+	)
+	(gr_text "+"
+		(at 87.7 58.45 0)
+		(layer "F.SilkS")
+		(effects
+			(font
+				(size 1.2 1.2)
+				(thickness 0.15)
+			)
+		)
+	)
+	(gr_text "-"
+		(at 87.7 63.53 0)
+		(layer "F.SilkS")
+		(effects
+			(font
+				(size 1.2 1.2)
+				(thickness 0.15)
+			)
+		)
+	)
+	(gr_text "BOOT"
+		(at 49.5 58.5 0)
+		(layer "B.SilkS")
+		(effects
+			(font
+				(size 1 1)
+				(thickness 0.15)
+			)
+			(justify mirror)
+		)
+	)
+	(gr_text "MCU RST"
+		(at 65 64.599999 0)
+		(layer "B.SilkS")
+		(effects
+			(font
+				(size 1 1)
+				(thickness 0.15)
+			)
+			(justify mirror)
+		)
+	)
+	(gr_text "RACK ATX R3"
+		(at 60 40 0)
+		(layer "B.SilkS")
+		(effects
+			(font
+				(size 1.2 1.2)
+				(thickness 0.15)
+			)
+			(justify mirror)
+		)
+	)
