File: hardware/cad/B2/host01.kicad_sch (KiCad schematic)
At the start: 19 parts, among them J01 S10B-PHDSS(LF)(SN), Q5 MMBT3904, Q6 MMBT3904, U8 TLP3122A(TPL,E, U9 TLP3122A(TPL,E

Commit message: Update Site source
Parts:
- D2, D3: LCSC C2841440 -> C5451656
