File: hardware/cad/B2/host02.kicad_sch (KiCad schematic)
At the start: 19 parts, among them J02 S10B-PHDSS(LF)(SN), Q7 MMBT3904, Q8 MMBT3904, U10 TLP3122A(TPL,E, U11 TLP3122A(TPL,E

Commit message: Update Site source
Parts:
- D4, D5: LCSC C2841440 -> C5451656
