File: hardware/cad/B2/host03.kicad_sch (KiCad schematic)
At the start: 19 parts, among them J03 S10B-PHDSS(LF)(SN), Q10 MMBT3904, Q9 MMBT3904, U12 TLP3122A(TPL,E, U13 TLP3122A(TPL,E

Commit message: Update Site source
Parts:
- D6, D7: LCSC C2841440 -> C5451656
