File: hardware/cad/B2/host04.kicad_sch (KiCad schematic)
At the start: 19 parts, among them J04 S10B-PHDSS(LF)(SN), Q11 MMBT3904, Q12 MMBT3904, U14 TLP3122A(TPL,E, U15 TLP3122A(TPL,E

Commit message: Update Site source
Parts:
- D8, D9: LCSC C2841440 -> C5451656
