File: hardware/cad/B2/host05.kicad_sch (KiCad schematic)
At the start: 19 parts, among them J05 S10B-PHDSS(LF)(SN), Q13 MMBT3904, Q14 MMBT3904, U16 TLP3122A(TPL,E, U17 TLP3122A(TPL,E

Commit message: Update Site source
Parts:
- D10, D11: LCSC C2841440 -> C5451656
