File: hardware/cad/B2/host06.kicad_sch (KiCad schematic)
At the start: 19 parts, among them J06 S10B-PHDSS(LF)(SN), Q15 MMBT3904, Q16 MMBT3904, U18 TLP3122A(TPL,E, U19 TLP3122A(TPL,E

Commit message: Update Site source
Parts:
- D12, D13: LCSC C2841440 -> C5451656
