File: hardware/cad/B2/host07.kicad_sch (KiCad schematic)
At the start: 19 parts, among them J07 S10B-PHDSS(LF)(SN), Q17 MMBT3904, Q18 MMBT3904, U20 TLP3122A(TPL,E, U21 TLP3122A(TPL,E

Commit message: Update Site source
Parts:
- D14, D15: LCSC C2841440 -> C5451656
