File: hardware/cad/B2/host08.kicad_sch (KiCad schematic)
At the start: 19 parts, among them J08 S10B-PHDSS(LF)(SN), Q19 MMBT3904, Q20 MMBT3904, U22 TLP3122A(TPL,E, U23 TLP3122A(TPL,E

Commit message: Update Site source
Parts:
- D16, D17: LCSC C2841440 -> C5451656
