File: hardware/cad/B2/host09.kicad_sch (KiCad schematic)
At the start: 19 parts, among them J09 S10B-PHDSS(LF)(SN), Q21 MMBT3904, Q22 MMBT3904, U24 TLP3122A(TPL,E, U25 TLP3122A(TPL,E

Commit message: Update Site source
Parts:
- D18, D19: LCSC C2841440 -> C5451656
