File: hardware/cad/B2/host10.kicad_sch (KiCad schematic)
At the start: 19 parts, among them J10 S10B-PHDSS(LF)(SN), Q23 MMBT3904, Q24 MMBT3904, U26 TLP3122A(TPL,E, U27 TLP3122A(TPL,E

Commit message: Update Site source
Parts:
- D20, D21: LCSC C2841440 -> C5451656
